Commit message: Update bveeta_shape.urdf
changes stl file from bveeta.stl to bveeta_base.stl

File: Source_code/urdf_bveeta/bveeta_shape.urdf (robot description, URDF)
Before this commit: robot bveeta_mini, 2 links, 1 joints
Links:
- link base_link: geometry visual mesh filename=package://urdf_bveeta/meshes/bveeta_base.stl scale=0.001 0.001 0.001

Commit message: Update bveeta_shape.urdf
change bveeta_base.stl to bveeta.stl

File: Source_code/urdf_bveeta/bveeta_shape.urdf (robot description, URDF)
Before this commit: robot bveeta_mini, 2 links, 1 joints
Links:
- link base_link: geometry visual mesh filename=package://urdf_bveeta/meshes/bveeta.stl scale=0.001 0.001 0.001
